File: Air_Piston_Oil_Control/Air_Piston_Oil_Control.kicad_sch (KiCad schematic)
At the start: 51 parts, among them J1 Conn_01x20_Pin, J2 Conn_02x06_Odd_Even, Q1 NTR4003NT3G, Q2 NTR4003NT3G, U1 STM32G431RBT6, U2 AMS1117-3.3, U4 LTL-30EHJH96, U5 MAX6817EUT_T, U6 CPC1966YX6, U7 CPC1966YX6, U8 CPC1966YX6, U9 CPC1966YX6, Y1 X322524MSB4SI

Commit message: Ver B manufacturing, removed solder pads
Parts:
- removed JP1, JP10, JP11, JP12, JP13, JP14, JP15, JP2, JP3, JP4, JP5, JP6, JP7, JP8, JP9: SolderJumper_2_Open, Jumper:SolderJumper-2_P1.3mm_Open_Pad1.0x1.5mm, symbol Jumper:SolderJumper_2_Open
- C10, C12, C14, C18, C7, C8, C9: value 100n -> 100nF
- C11: value 4.7u -> 4.7uF
- C13, C15: value 1u -> 1uF
- C16, C17: value 6.8p -> 6.8pF
- R2, R3, R4, R5: value 1K -> 1k
Connections:
- net AC1/OVERHEAT_LED: now also U1.9 (PC1)
- net DEMAG_IN: now also U1.23 (PC5)
- net DEMAG_MOSFET: now also U1.20 (PA6)
- net MACHINE_LED: now also U1.18 (PA4)
- net MAG_IN: now also U1.22 (PC4)
- net MAG_MOSFET: now also U1.19 (PA5)
- net SIG_CLAMP: now also U1.17 (PA3)
- net SIG_OILER: now also U1.12 (PA0)
- net SIG_SOLENOID1: now also U1.14 (PA2)
- net SIG_SOLENOID2: now also U1.13 (PA1)
- net SPRAY_TIME/S5: now also U1.8 (PC0)
- net TEMP_SENS1: now also U1.10 (PC2)
- net TEMP_SENS2: now also U1.11 (PC3)
- net at U1.5 (PF0): now also C16.1, Y1.1
- net at U1.6 (PF1): now also C17.1, Y1.3
